File: displaycontrol.sch (EAGLE design)
At the start: 49 parts, among them IC1 25LC080SN, J1 GRPB052VWQS-RC, J2 5.5x2.1mm Barrel, J3 98424-F52, Q1 MMPQ3904, U1 LPC1315FBD48,551, U2 ADP3300ARTZ-3.3RL7, U3 UDN2987LWTR-6-T, U4 UDN2987LWTR-6-T, Y1 12MHz

Commit message: changed trans
Parts:
- removed D1, D2, D3, D4, D5, D6, D7, D8: MMSD4148, adafruit:DIODESOD-123
- added Q2, Q3, Q4, Q5: MMBT3904, SparkFun-DiscreteSemi:TRANSISTOR_NPNMMBT2222A
- R2, R3, R4, R5: value 4.7k -> 2.7k
- R6, R7, R8, R9: value 14 -> 10
Connections:
- removed net N$10: Q1.E1, R6.1
- removed net N$11: D5.A, Q1.B3, R4.2
- removed net N$12: D5.C, D6.A
- removed net N$14: D7.A, Q1.B4, R5.2
- removed net N$15: D7.C, D8.A
- removed net N$17: Q1.E2, R7.1
- removed net N$19: Q1.E3, R8.1
- removed net N$21: Q1.E4, R9.1
- removed net N$5: D1.A, Q1.B1, R2.2
- removed net N$8: D3.A, Q1.B2, R3.2
- removed net N$9: D3.C, D4.A
- new net COLCTRL_1: Q1.B4, Q5.C, R5.2
- new net COLCTRL_2: Q1.B3, Q4.C, R4.2
- new net COLCTRL_3: Q1.B2, Q3.C, R3.2
- new net COLCTRL_A: Q1.B1, Q2.C, R2.2
- new net EMITCTRL_1: Q1.E4, Q5.B, R9.1
- new net EMITCTRL_2: Q1.E3, Q4.B, R8.1
- new net EMITCTRL_3: Q1.E2, Q3.B, R7.1
- new net EMITCTRL_A: Q1.E1, Q2.B, R6.1
- net GND: now also Q2.E, Q3.E, Q4.E, Q5.E; no longer D2.C, D4.C, D6.C, D8.C
- net N$6: now also U1.PIO0_23/AD7; no longer D1.C, D2.A
Other:
- moved on the sheet: R1, R10, R11, R12, R13, R6, R7, R8, R9
